File: PCB_GIRLS_DAY/PCB_GIRLS_DAY.kicad_sch (KiCad schematic)
At the start: 6 parts

Commit message: Kicad - PCB avant routage
Other:
- note added: "Power LED"
Changed lines of the file:
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@@
+		)
+	)
+	(rectangle
+		(start 15.24 139.7)
+		(end 76.2 196.85)
+		(stroke
+			(width 0.254)
+			(type dash)
+		)
+		(fill
+			(type none)
 		)
 	)
@@
 		(effects
 			(font
+				(size 2.54 2.54)
+				(thickness 0.508)
+				(bold yes)
+			)
+		)
+	)
+	(text "Power LED\n"
+		(exclude_from_sim no)
+		(at 27.94 143.256 0)
+		(effects
+			(font
