File: PCB_GIRLS_DAY/PCB_GIRLS_DAY.kicad_sch (KiCad schematic)
At the start: 6 parts

Commit message: PCB_Update
Other:
- sheet SCH_MCU ports: added none; removed PC9
- sheet SCH_PINOUT ports: added none; removed PC9
Changed lines of the file:
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@@
-			)
-		)
-		(pin "PC9" input
-			(at 147.32 110.49 180)
-			(effects
-				(font
-					(size 1.27 1.27)
-				)
-				(justify left)
 			)
 		)
@@
 			(effects
 				(font
-					(size 1.27 1.27)
-				)
-				(justify right)
-			)
-		)
-		(pin "PC9" output
-			(at 135.89 110.49 0)
-			(effects
-				(font

Commit message: PCB revision Cyprien
Parts:
- added H2, H3, H4, H5: MountingHole, MountingHole:MountingHole_2.1mm, symbol Mechanical:MountingHole
Other:
- sheet SCH_MCU ports: added PB12, PB13, PB15; removed PA4, PA5, PB0, PB1, PB2, PB3, PB4, PB8, PC0, PC1, PC10, PC11, PC12, PC14, PC2, PC3, PC4, PC5
- sheet SCH_PINOUT ports: added PB12, PB13, PB15; removed PA4, PA5, PB0, PB1, PB2, PB3, PB4, PB8, PC0, PC1, PC10, PC11, PC12, PC14, PC2, PC3, PC4, PC5
