File: PCB_GIRLS_DAY/SCH_FS1000.kicad_sch (KiCad schematic)
At the start: 38 parts, among them Q1 S8050, Q2 2SC3357-T1-A, Q3 MMBT918, U5 SB7343392TT, U6 LM358_C5252902

Commit message: Kicad - PCB avant routage
Parts:
- C16: footprint EasyEDA:C0603 -> Capacitor_SMD:C_0603_1608Metric
- C17, C21, C22: footprint EasyEDA:C0603 -> Capacitor_SMD:C_0603_1608Metric_Pad1.08x0.95mm_HandSolder
Changed lines of the file:
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@@
 			)
 		)
-		(property "Footprint" "EasyEDA:C0603"
+		(property "Footprint" "Capacitor_SMD:C_0603_1608Metric_Pad1.08x0.95mm_HandSolder"
 			(at 134.62 81.28 0)
 			(hide yes)
@@
 			)
 		)
-		(property "Footprint" "EasyEDA:C0603"
+		(property "Footprint" "Capacitor_SMD:C_0603_1608Metric_Pad1.08x0.95mm_HandSolder"
 			(at 123.19 97.79 0)
 			(hide yes)
@@
 			)
 		)
-		(property "Footprint" "EasyEDA:C0603"
+		(property "Footprint" "Capacitor_SMD:C_0603_1608Metric"
 			(at 39.37 69.85 0)
 			(hide yes)
@@
 			)
 		)
-		(property "Footprint" "EasyEDA:C0603"
+		(property "Footprint" "Capacitor_SMD:C_0603_1608Metric_Pad1.08x0.95mm_HandSolder"
 			(at 87.63 63.5 0)
 			(hide yes)
@@
 		)
 		(property "Footprint" "EasyEDA:DO-35_BD2.0-L4.2-P8.20-D0.5-RD"
-			(at 166.37 91.44 0)
+			(at 167.132 92.71 0)
 			(hide yes)
 			(show_name no)
