File: PCB_GIRLS_DAY/SCH_FS1000.kicad_sch (KiCad schematic)
At the start: 38 parts, among them Q1 S8050, Q2 2SC3357-T1-A, Q3 MMBT918, U5 SB7343392TT, U6 LM358_C5252902

Commit message: PCB_Update
Parts:
- removed L2: 3turns, symbol Device:L
- removed L3: 8turns, symbol Device:L
- removed L4: 1.5 turns, symbol Device:L
- added L6: 180nH, EasyEDA:IND-SMD_L1.8-W1.2, symbol EasyEDA:AISC-0603-R18J-T
- added L7: 36nH, EasyEDA:IND-SMD_L1.0-W0.5-2, symbol EasyEDA:LQW15AN36NG00D
- added L8: 15nH, EasyEDA:IND-SMD_L1.0-W0.5-2, symbol EasyEDA:LQW15AN15NG00D
- AE1, AE2: footprint (none) -> Connector_Wire:SolderWire-2.5sqmm_1x01_D2.4mm_OD4.4mm
Connections:
- net +5V: now also L6.1
- net at C18.1, C22.2, R15.1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: now also L8.2
- net at C16.2, R9.1, U5.1: now also L6.2, L7.1
- net at AE2.1 (A), C21.2, C22.1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: now also L8.1
- net at C17.2, Q2.2 (C): now also L7.2

Commit message: PCB revision Cyprien
Parts:
- removed U5: SB7343392TT, EasyEDA:CRYSTAL-SMD_3P-L7.7-W3.7-P2.50_SB7343392TT, symbol EasyEDA:SB7343392TT
- added L2, L3: BW433MNX1304, EasyEDA:ANT-SMD_L130-W42_BW433MNX, symbol EasyEDA:BW433MNX1304
- added Y1: Crystal_GND3, Package_TO_SOT_THT:TO-39-3, symbol Device:Crystal_GND3
- AE1, AE2: footprint Connector_Wire:SolderWire-2.5sqmm_1x01_D2.4mm_OD4.4mm -> Connector_Samtec_HPM_THT:Samtec_HPM-01-01-x-S_Straight_1x01_Pitch5.08mm
Connections:
- net GND: now also Y1.3
- net at C16.2, L6.2, L7.1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: now also Y1.2
- net at Q2.1 (B), R9.2: now also Y1.1
- net at AE2.1 (A), C21.2, C22.1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: now also L3.2 (ANT)
- net at AE1.1 (A), C17.1: now also L2.2 (ANT)
- no-connect marks 0 -> 2
