File: PCB_GIRLS_DAY/SCH_MCU.kicad_sch (KiCad schematic)
At the start: 24 parts, among them J1 USB_B_Micro, J2 Conn_01x04_Pin, SW1 SW_SPDT, U1 STM32F446RETx, X1 X50328MSB2GI

Commit message: Kicad - PCB avant routage
Parts:
- removed L1: L_Ferrite, symbol Device:L_Ferrite
- added L1: FCM1608KF-601T05, EasyEDA:L0603, symbol EasyEDA:FCM1608KF-601T05
- added R21: 0Ω, PCM_JLCPCB:R_0603, symbol PCM_JLCPCB-Resistors:0603,0Ω
- J1: footprint (none) -> Connector_USB:USB_Micro-B_Wuerth_629105150521
- J2: footprint (none) -> Connector_PinHeader_2.54mm:PinHeader_1x04_P2.54mm_Vertical
- SW1: footprint (none) -> Button_Switch_THT:SW_E-Switch_EG1224_SPDT_Angled
Connections:
- net +3.3VA: now also L1.2
- net +3V3: now also L1.1
- net GND: now also R21.1
- net PB2: now also R21.2
Other:
- note added: "BOOT MODES"
- moved on the sheet: C2
