File: PCB_GIRLS_DAY/SCH_MCU.kicad_sch (KiCad schematic)
At the start: 25 parts, among them J1 USB_B_Micro, J2 Conn_01x04_Pin, SW1 SW_SPDT, U1 STM32F446RETx, X1 X50328MSB2GI

Commit message: PCB_Update
Parts:
- SW1: footprint Button_Switch_THT:SW_E-Switch_EG1224_SPDT_Angled -> Button_Switch_SMD:SW_SPDT_PCM12
Connections:
- net PC9: no longer names the net of U1.40 (PC9)
- no-connect marks 8 -> 10
Changed lines of the file:
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@@
 	)
 	(no_connect
+		(at 52.07 102.87)
+	)
+	(no_connect
 		(at 118.11 82.55)
 	)
@@
 	)
 	(no_connect
+		(at 99.06 95.25)
+	)
+	(no_connect
 		(at 99.06 125.73)
 	)
@@
 		)
 	)
-	(hierarchical_label "PC9"
-		(shape input)
-		(at 52.07 102.87 180)
-		(effects
-			(font
-				(size 1.27 1.27)
-			)
-			(justify right)
-		)
-	)
 	(hierarchical_label "PB6"
 		(shape input)
@@
 			)
 		)
-		(property "Footprint" "Button_Switch_THT:SW_E-Switch_EG1224_SPDT_Angled"
+		(property "Footprint" "Button_Switch_SMD:SW_SPDT_PCM12"
 			(at 25.4 62.23 0)
 			(hide yes)

Commit message: PCB revision Cyprien
Parts:
- removed J2: Conn_01x04_Pin, Connector_PinHeader_2.54mm:PinHeader_1x04_P2.54mm_Vertical, symbol Connector:Conn_01x04_Pin
- added J2: Conn_02x05_Counter_Clockwise, Connector:Tag-Connect_TC2050-IDC-FP_2x05_P1.27mm_Vertical, symbol Connector_Generic:Conn_02x05_Counter_Clockwise
- added R22: 1.5kΩ, PCM_JLCPCB:R_0603, symbol PCM_JLCPCB-Resistors:0603,1.5kΩ
- added R23, R25, R26: 22Ω, PCM_JLCPCB:R_0603, symbol PCM_JLCPCB-Resistors:0603,22Ω
Connections:
- net +3V3: now also J2.1 (Pin_1), R22.1
- net GND: now also J1.SH (Shield), J2.3 (Pin_3)
- net NRST: now also R26.1
- net SWCLK: now also R23.1
- net SWDIO: now also R25.1
- net PB12: now reaches U1.33 (PB12)
- net PB13: now reaches U1.34 (PB13)
- net PB15: now reaches U1.36 (PB15)
- net PA4: no longer names the net of U1.20 (PA4)
- net PA5 renamed LED
- net PB0: no longer names the net of U1.26 (PB0)
- net PB1: no longer names the net of U1.27 (PB1)
- net PB2: no longer names the net of R21.2, U1.28 (PB2)
- net PB3: no longer names the net of U1.55 (PB3)
- net PB4: no longer names the net of U1.56 (PB4)
- net PB8: no longer names the net of U1.61 (PB8)
- net PC0: no longer names the net of U1.8 (PC0)
- net PC1: no longer names the net of U1.9 (PC1)
- net PC10: no longer names the net of U1.51 (PC10)
- net PC11: no longer names the net of U1.52 (PC11)
- net PC12: no longer names the net of U1.53 (PC12)
- net PC14: no longer names the net of U1.3 (PC14)
- net PC2: no longer names the net of U1.10 (PC2)
- net PC3: no longer names the net of U1.11 (PC3)
- net PC4: no longer names the net of U1.24 (PC4)
- net PC5: no longer names the net of U1.25 (PC5)
- net USB_D+ renamed USB_DP
- net USB_DP: now also R22.2
- net USB_D- renamed USB_DN
- new net: J2.2 (Pin_2), R23.2
- new net: J2.4 (Pin_4), R25.2
- new net: J2.5 (Pin_5), R26.2
- no-connect marks 10 -> 27
Other:
- moved on the sheet: J1
