File: PCB_GIRLS_DAY/SCH_PINOUT.kicad_sch (KiCad schematic)
At the start: 2 parts, among them J4 Conn_01x03_Pin, J5 Conn_02x20_Odd_Even

Commit message: Kicad - PCB avant routage
Parts:
- J4: footprint (none) -> Connector_PinHeader_2.54mm:PinHeader_1x03_P2.54mm_Vertical
- J5: footprint (none) -> Connector_PinHeader_2.54mm:PinHeader_2x20_P2.54mm_Vertical
Changed lines of the file:
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@@
 			)
 		)
-		(property "Footprint" ""
+		(property "Footprint" "Connector_PinHeader_2.54mm:PinHeader_1x03_P2.54mm_Vertical"
 			(at 116.84 99.06 0)
 			(hide yes)
@@
 			)
 		)
-		(property "Footprint" ""
+		(property "Footprint" "Connector_PinHeader_2.54mm:PinHeader_2x20_P2.54mm_Vertical"
 			(at 170.18 102.87 0)
 			(hide yes)
