File: PCB_GIRLS_DAY/SCH_PINOUT.kicad_sch (KiCad schematic)
At the start: 2 parts, among them J4 Conn_01x03_Pin, J5 Conn_02x20_Odd_Even

Commit message: PCB_Update
Connections:
- net PC9: no longer names the net of J5.30 (Pin_30)
- no-connect marks 0 -> 1
Changed lines of the file:
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@@
 		)
+	)
+	(no_connect
+		(at 181.61 115.57)
 	)
 	(wire
@@
 		(effects
 			(font
-				(size 1.27 1.27)
-			)
-			(justify left)
-		)
-	)
-	(hierarchical_label "PC9"
-		(shape output)
-		(at 181.61 115.57 0)
-		(effects
-			(font

Commit message: PCB revision Cyprien
Parts:
- removed J5: Conn_02x20_Odd_Even, Connector_PinHeader_2.54mm:PinHeader_2x20_P2.54mm_Vertical, symbol Connector_Generic:Conn_02x20_Odd_Even
- added J6: Conn_02x12_Odd_Even, Connector_Samtec_HLE_THT:Samtec_HLE-112-02-xx-DV-TE_2x12_P2.54mm_Horizontal, symbol Connector_Generic:Conn_02x12_Odd_Even
Connections:
- net +3V3: now also J6.23 (Pin_23)
- net +5V: now also J6.24 (Pin_24)
- net +E5V: now also J6.2 (Pin_2)
- net +U5V: now also J6.1 (Pin_1)
- net GND: now also J6.21 (Pin_21), J6.22 (Pin_22), J6.3 (Pin_3), J6.4 (Pin_4)
- net PA0: now also J6.19 (Pin_19)
- net PA1: now also J6.17 (Pin_17)
- net PA2: now also J6.15 (Pin_15)
- net PA3: now also J6.13 (Pin_13)
- net PA8: now also J6.12 (Pin_12)
- net PA9: now also J6.11 (Pin_11)
- net PB14: now also J6.18 (Pin_18)
- net PB5: now also J6.10 (Pin_10)
- net PB6: now also J6.6 (Pin_6)
- net PB7: now also J6.8 (Pin_8)
- net PC6: now also J6.5 (Pin_5)
- net PC7: now also J6.7 (Pin_7)
- net PC8: now also J6.9 (Pin_9)
- new net PB12: J6.14 (Pin_14)
- new net PB13: J6.16 (Pin_16)
- new net PB15: J6.20 (Pin_20)
- no-connect marks 1 -> 0
