File: pcb/sch_fs1000.kicad_sch (KiCad schematic)
At the start: 40 parts, among them J5 Conn_01x03_Pin, J7 Conn_01x04_Pin, Q1 S8050, Q2 2SC3357-T1-A, Q3 MMBT918, U6 LM358_C5252902, Y1 Crystal_GND3

Commit message: fix(layout): footprints
Parts:
- AE1, AE2: footprint Connector_PinHeader_1.00mm:PinHeader_1x01_P1.00mm_Vertical -> library:AntennaHole
- L5: footprint EasyEDA:IND-SMD_L10.2-W10.2-LS10.8 -> Inductor_SMD:L_0805_2012Metric
- L6: footprint EasyEDA:IND-SMD_L1.8-W1.2 -> Inductor_SMD:L_0603_1608Metric
- L7, L8: footprint EasyEDA:IND-SMD_L1.0-W0.5-2 -> Inductor_SMD:L_0603_1608Metric
Changed lines of the file:
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@@
 			)
 		)
-		(property "Footprint" "EasyEDA:IND-SMD_L1.0-W0.5-2"
+		(property "Footprint" "Inductor_SMD:L_0603_1608Metric"
 			(at 63.5 64.77 0)
 			(hide yes)
@@
 			)
 		)
-		(property "Footprint" "Connector_PinHeader_1.00mm:PinHeader_1x01_P1.00mm_Vertical"
+		(property "Footprint" "library:AntennaHole"
 			(at 116.84 59.69 0)
 			(hide yes)
@@
 			)
 		)
-		(property "Footprint" "Connector_PinHeader_1.00mm:PinHeader_1x01_P1.00mm_Vertical"
+		(property "Footprint" "library:AntennaHole"
 			(at 99.06 59.69 0)
 			(hide yes)
@@
 			)
 		)
-		(property "Footprint" "EasyEDA:IND-SMD_L1.0-W0.5-2"
+		(property "Footprint" "Inductor_SMD:L_0603_1608Metric"
 			(at 134.62 69.85 0)
 			(hide yes)
@@
 			)
 		)
-		(property "Footprint" "EasyEDA:IND-SMD_L10.2-W10.2-LS10.8"
+		(property "Footprint" "Inductor_SMD:L_0805_2012Metric"
 			(at 134.62 110.49 0)
 			(hide yes)
@@
 			)
 		)
-		(property "Footprint" "EasyEDA:IND-SMD_L1.8-W1.2"
+		(property "Footprint" "Inductor_SMD:L_0603_1608Metric"
 			(at 50.8 64.77 0)
 			(hide yes)

Commit message: feat(layout): component placement
Parts:
- added JP2, JP3, JP4, JP5: SolderJumper_2_Bridged, Jumper:SolderJumper-2_P1.3mm_Bridged_RoundedPad1.0x1.5mm, symbol Jumper:SolderJumper_2_Bridged
- C21: footprint Capacitor_SMD:C_0603_1608Metric_Pad1.08x0.95mm_HandSolder -> Capacitor_SMD:C_0603_1608Metric
Connections:
- net +5V: now also J7.4 (Pin_4), JP3.1 (A), JP5.1 (A); no longer C23.1, J7.1 (Pin_1), L6.1, R11.1, R16.2, U6.8 (VCC)
- net GND: now also J5.1 (Pin_1), J7.1 (Pin_1); no longer J5.3 (Pin_3), J7.4 (Pin_4)
- net DATA IN renamed DATA_IN
- net DATA_IN: now also JP4.1 (A); no longer U6.7 (OUT2)
- net DATA OUT renamed DATA_OUT_FS
- net DATA_OUT_FS: now also JP2.2 (B); no longer J5.1 (Pin_1)
- new net 5V_FS: JP3.2 (B), L6.1
- new net 5V_XY: C23.1, JP5.2 (B), R11.1, R16.2, U6.8 (VCC)
- new net DATA_IN_XY: JP4.2 (B), U6.7 (OUT2)
- new net DATA_OUT: J5.3 (Pin_3), JP2.1 (A)
Other:
- moved on the sheet: J5, J7
