File: pcb/sch_mcu.kicad_sch (KiCad schematic)
At the start: 32 parts, among them J1 Conn_01x03_Pin, J3 USB_C_Receptacle_USB2.0_14P, J8 Conn_ARM_JTAG_SWD_10, SW1 SW_Push_WE, SW3 SW_Push_WE, U1 STM32F446RETx, U4 USBLC6-4SC6, Y2 Crystal_4-pin

Commit message: fix(layout): footprints
Parts:
- removed J1: Conn_01x03_Pin, Connector_PinHeader_2.54mm:PinHeader_1x03_P2.54mm_Vertical, symbol Connector:Conn_01x03_Pin
- added JP1: SolderJumper_2_Bridged, Jumper:SolderJumper-2_P1.3mm_Bridged_RoundedPad1.0x1.5mm, symbol Jumper:SolderJumper_2_Bridged
- added SW4: SW_Push_WE, library:SW_Tactile_SPST_Angled_WE, symbol library:SW_Push_WE
Connections:
- net +3V3: now also SW4.2
- net GND: now also R7.2, JP1.1 (A); no longer J8.3 (GND), J8.5 (GND)
- net at R7.1, U1.60 (BOOT0): now also SW4.3
- new net: J8.3 (GND), J8.5 (GND), JP1.2 (B)
Other:
- moved on the sheet: R7

Commit message: feat(layout): component placement
Parts:
- added C12, C15: 1uF, Capacitor_SMD:C_0603_1608Metric, symbol PCM_JLCPCB-Capacitors:0603,1uF
- C5, C6, C7, C8: footprint PCM_JLCPCB:C_0603 -> Capacitor_SMD:C_0603_1608Metric
Connections:
- net +3V3: now also SW4.3, C12.1, C15.1; no longer SW4.2
- net GND: now also C12.2, C15.2
- net at R7.1, U1.60 (BOOT0): now also SW4.2; no longer SW4.3
