File: pcb/sch_pinout.kicad_sch (KiCad schematic)
At the start: 2 parts, among them J4 Conn_01x03_Pin, J6 Conn_02x12_Odd_Even

Commit message: feat(sch): schematic review
Parts:
- J4: footprint Connector_PinHeader_2.54mm:PinHeader_1x03_P2.54mm_Vertical -> Connector_JST:JST_XA_B03B-XASK-1-A_1x03_P2.50mm_Vertical
Changed lines of the file:
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@@
 		)
 		(instances
-			(project "PCB_GIRLS_DAY"
+			(project "enclosure_pcb"
 				(path "/4a16a4d9-4fe7-4c30-8337-203b926a87e2/b67f4f69-488b-4c78-b1eb-3899eb6aef9b"
 					(reference "#PWR069")
@@
 		)
 		(instances
-			(project "PCB_GIRLS_DAY"
+			(project "enclosure_pcb"
 				(path "/4a16a4d9-4fe7-4c30-8337-203b926a87e2/b67f4f69-488b-4c78-b1eb-3899eb6aef9b"
 					(reference "#PWR067")
@@
 		)
 		(instances
-			(project "PCB_GIRLS_DAY"
+			(project "enclosure_pcb"
 				(path "/4a16a4d9-4fe7-4c30-8337-203b926a87e2/b67f4f69-488b-4c78-b1eb-3899eb6aef9b"
 					(reference "#PWR046")
@@
 		)
 		(instances
-			(project "PCB_GIRLS_DAY"
+			(project "enclosure_pcb"
 				(path "/4a16a4d9-4fe7-4c30-8337-203b926a87e2/b67f4f69-488b-4c78-b1eb-3899eb6aef9b"
 					(reference "#PWR065")
@@
 		)
 		(instances
-			(project "PCB_GIRLS_DAY"
+			(project "enclosure_pcb"
 				(path "/4a16a4d9-4fe7-4c30-8337-203b926a87e2/b67f4f69-488b-4c78-b1eb-3899eb6aef9b"
 					(reference "#PWR047")
@@
 		)
 		(instances
-			(project "PCB_GIRLS_DAY"
+			(project "enclosure_pcb"
 				(path "/4a16a4d9-4fe7-4c30-8337-203b926a87e2/b67f4f69-488b-4c78-b1eb-3899eb6aef9b"
 					(reference "#PWR064")
@@
 			)
 		)
-		(property "Footprint" "Connector_PinHeader_2.54mm:PinHeader_1x03_P2.54mm_Vertical"
+		(property "Footprint" "Connector_JST:JST_XA_B03B-XASK-1-A_1x03_P2.50mm_Vertical"
 			(at 116.84 99.06 0)
 			(hide yes)
@@
 		)
 		(instances
-			(project "PCB_GIRLS_DAY"
+			(project "enclosure_pcb"
 				(path "/4a16a4d9-4fe7-4c30-8337-203b926a87e2/b67f4f69-488b-4c78-b1eb-3899eb6aef9b"
 					(reference "J4")
@@
 		)
 		(instances
-			(project "PCB_GIRLS_DAY"
+			(project "enclosure_pcb"
 				(path "/4a16a4d9-4fe7-4c30-8337-203b926a87e2/b67f4f69-488b-4c78-b1eb-3899eb6aef9b"
 					(reference "#PWR071")
@@
 		)
 		(instances
-			(project "PCB_GIRLS_DAY"
+			(project "enclosure_pcb"
 				(path "/4a16a4d9-4fe7-4c30-8337-203b926a87e2/b67f4f69-488b-4c78-b1eb-3899eb6aef9b"
 					(reference "J6")
@@
 		)
 		(instances
-			(project "PCB_GIRLS_DAY"
+			(project "enclosure_pcb"
 				(path "/4a16a4d9-4fe7-4c30-8337-203b926a87e2/b67f4f69-488b-4c78-b1eb-3899eb6aef9b"
 					(reference "#PWR070")
@@
 		)
 		(instances
-			(project "PCB_GIRLS_DAY"
+			(project "enclosure_pcb"
 				(path "/4a16a4d9-4fe7-4c30-8337-203b926a87e2/b67f4f69-488b-4c78-b1eb-3899eb6aef9b"
 					(reference "#PWR068")
@@
 		)
 		(instances
-			(project "PCB_GIRLS_DAY"
+			(project "enclosure_pcb"
 				(path "/4a16a4d9-4fe7-4c30-8337-203b926a87e2/b67f4f69-488b-4c78-b1eb-3899eb6aef9b"
 					(reference "#PWR066")

Commit message: V2_avant_revision
Connections:
- net PA0: now also J6.15 (Pin_15); no longer J6.19 (Pin_19)
- net PA2: now also J6.19 (Pin_19); no longer J6.15 (Pin_15)
- net PC6: now also J6.9 (Pin_9); no longer J6.5 (Pin_5)
- net PC8: now also J6.5 (Pin_5); no longer J6.9 (Pin_9)
Changed lines of the file:
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@@
-		)
-	)
-	(hierarchical_label "PC6"
-		(shape output)
-		(at 162.56 91.44 180)
-		(effects
-			(font
-				(size 1.27 1.27)
-			)
-			(justify right)
 		)
 	)
@@
 		(shape output)
 		(at 162.56 106.68 180)
+		(effects
+			(font
+				(size 1.27 1.27)
+			)
+			(justify right)
+		)
+	)
+	(hierarchical_label "PC8"
+		(shape output)
+		(at 162.56 91.44 180)
 		(effects
 			(font
@@
 		)
 	)
-	(hierarchical_label "PA0"
-		(shape output)
-		(at 162.56 109.22 180)
-		(effects
-			(font
-				(size 1.27 1.27)
-			)
-			(justify right)
-		)
-	)
 	(hierarchical_label "PB7"
 		(shape output)
@@
 		)
 	)
+	(hierarchical_label "PC6"
+		(shape output)
+		(at 162.56 96.52 180)
+		(effects
+			(font
+				(size 1.27 1.27)
+			)
+			(justify right)
+		)
+	)
 	(hierarchical_label "PA2"
+		(shape output)
+		(at 162.56 109.22 180)
+		(effects
+			(font
+				(size 1.27 1.27)
+			)
+			(justify right)
+		)
+	)
+	(hierarchical_label "PA0"
 		(shape output)
 		(at 162.56 104.14 180)
@@
 		)
 	)
-	(hierarchical_label "PC8"
-		(shape output)
-		(at 162.56 96.52 180)
-		(effects
-			(font
-				(size 1.27 1.27)
-			)
-			(justify right)
-		)
-	)

Commit message: fix(layout): footprints
Parts:
- J4: footprint Connector_JST:JST_XA_B03B-XASK-1-A_1x03_P2.50mm_Vertical -> Connector_JST:JST_XH_B3B-XH-A_1x03_P2.50mm_Vertical
Changed lines of the file:
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@@
 			)
 		)
-		(property "Footprint" "Connector_JST:JST_XA_B03B-XASK-1-A_1x03_P2.50mm_Vertical"
+		(property "Footprint" "Connector_JST:JST_XH_B3B-XH-A_1x03_P2.50mm_Vertical"
 			(at 116.84 99.06 0)
 			(hide yes)

Commit message: feat: pcb review
Parts:
- removed J6: Conn_02x12_Odd_Even, Connector_Samtec_HLE_THT:Samtec_HLE-112-02-xx-DV-TE_2x12_P2.54mm_Horizontal, symbol Connector_Generic:Conn_02x12_Odd_Even
