File: pcb/_restore_backup_2026-08-16T08-19-23-888/enclosure_pcb.kicad_pcb (KiCad board)
At the start: 2 copper layers, 100 x 80 mm, 102 parts, among them J3 USB_C_Receptacle_USB2.0_14P, J4 Conn_01x03_Pin, J5 Conn_01x03_Pin, J7 Conn_01x04_Pin, J8 Conn_ARM_JTAG_SWD_10, Q1 S8050, Q2 2SC3357-T1-A, Q3 MMBT918, SW1 SW_Push_WE, SW2 SW_Lever_RSPRO_5MS1, SW3 SW_Push_WE, SW4 SW_Push_WE, U1 STM32F446RETx, U2 LD1117S33TR_SOT223, U3 LD1117S50TR_SOT223, U4 USBLC6-4SC6, U6 LM358_C5252902, Y1 Crystal_GND3, Y2 Crystal_4-pin

Commit message: feat: pcb review
Parts:
- added J6: Conn_02x12_Odd_Even, Connector_Samtec_HLE_THT:Samtec_HLE-112-02-xx-DV-TE_2x12_P2.54mm_Horizontal, F.Cu at (105.0, 90.2)
- moved R4 4.00 mm to (133.0, 120.0)
- moved J4 2.61 mm to (108.5, 101.5)
- moved D1 2.25 mm to (150.0, 101.0)
- moved R1 2.25 mm to (146.0, 101.0)
- moved D2 2.00 mm to (150.0, 103.0)
- moved R2 2.00 mm to (146.0, 103.0)
- moved C8 2.00 mm to (129.0, 120.0)
- moved R5 2.00 mm to (131.0, 120.0)
- moved C10 1.00 mm to (132.5, 89.0)
- moved C11 1.00 mm to (132.5, 87.0)
- moved D4 0.50 mm to (150.0, 105.0)
- moved R6 0.50 mm to (146.0, 105.0)
Connections:
- J5 pad 3: /SCH_FS1000/DATA OUT -> /SCH_FS1000/DATA_OUT
- J7 pad 2: /SCH_FS1000/DATA IN -> /SCH_FS1000/DATA_IN
- J7 pad 3: /SCH_FS1000/DATA IN -> /SCH_FS1000/DATA_IN
- JP2 pad 1: /SCH_FS1000/DATA OUT -> /SCH_FS1000/DATA_OUT
- JP4 pad 1: /SCH_FS1000/DATA IN -> /SCH_FS1000/DATA_IN
- SW4 pad 1: GND -> unconnected-(SW4-Pad1)
- SW4 pad 4: GND -> unconnected-(SW4-Pad4)
- U1 pad 22: /SCH_FS1000/DATA IN -> /SCH_MCU/DATA_OUT
- U1 pad 23: /SCH_FS1000/DATA OUT -> /SCH_MCU/DATA_IN
Routing:
- net +3V3: track 219.8 -> 31.4 mm
- net +5V: track 181.5 -> 31.8 mm, vias 1 -> 0
- net +E5V: track 28.4 -> 128.9 mm
- net /SCH_FS1000/DATA IN: track 76.7 -> 0.00 mm
- net /SCH_MCU/NRST: track 78.0 -> 11.2 mm, vias 3 -> 0
- net /SCH_FS1000/DATA OUT: track 56.7 -> 0.00 mm
- net Net-(U1-BOOT0): track 68.5 -> 18.5 mm, vias 2 -> 0
- net +U5V: track 58.2 -> 98.3 mm
- net /SCH_MCU/PUSH_BTN: track 43.7 -> 13.2 mm, vias 2 -> 0
- net /SCH_MCU/PWM: track 28.5 -> 0.00 mm, vias 1 -> 0
- net /SCH_MCU/LED: track 28.1 -> 0.00 mm, vias 2 -> 0
- net /SCH_FS1000/DATA_IN: track 0.00 -> 8.47 mm
- net /SCH_FS1000/DATA_OUT: track 0.00 -> 3.54 mm
- net GND: vias 164 -> 74
