File: pcb/_restore_backup_2026-08-16T08-19-23-888/sch_mcu.kicad_sch (KiCad schematic)
At the start: 35 parts, among them J3 USB_C_Receptacle_USB2.0_14P, J8 Conn_ARM_JTAG_SWD_10, SW1 SW_Push_WE, SW3 SW_Push_WE, SW4 SW_Push_WE, U1 STM32F446RETx, U4 USBLC6-4SC6, Y2 Crystal_4-pin

Commit message: feat: pcb review
Connections:
- net GND: no longer SW4.1, SW4.4
Changed lines of the file:
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@@
 	)
 	(junction
-		(at 39.37 71.12)
-		(diameter 0)
-		(color 0 0 0 0)
-	)
-	(junction
 		(at 50.8 33.02)
 		(diameter 0)
@@
 	(wire
 		(pts
-			(xy 39.37 68.58) (xy 39.37 71.12)
-		)
-		(stroke
-			(width 0)
-			(type default)
-		)
-	)
-	(wire
-		(pts
 			(xy 46.99 115.57) (xy 58.42 115.57)
 		)
@@
 	(wire
 		(pts
-			(xy 36.83 68.58) (xy 39.37 68.58)
-		)
-		(stroke
-			(width 0)
-			(type default)
-		)
-	)
-	(wire
-		(pts
 			(xy 101.6 57.15) (xy 101.6 59.69)
 		)
@@
 	(wire
 		(pts
-			(xy 36.83 71.12) (xy 39.37 71.12)
-		)
-		(stroke
-			(width 0)
-			(type default)
-		)
-	)
-	(wire
-		(pts
 			(xy 58.42 33.02) (xy 58.42 36.83)
 		)
@@
 	(wire
 		(pts
-			(xy 39.37 71.12) (xy 41.91 71.12)
-		)
-		(stroke
-			(width 0)
-			(type default)
-		)
-	)
-	(wire
-		(pts
 			(xy 52.07 97.79) (xy 58.42 97.79)
 		)
@@
 					(unit 1)
 				)
-			)
-		)
-	)
-	(symbol
-		(lib_id "power:GND")
-		(at 41.91 71.12 90)
-		(unit 1)
-		(body_style 1)
-		(exclude_from_sim no)
-		(in_bom yes)
-		(on_board yes)
-		(in_pos_files yes)
-		(dnp no)
-		(fields_autoplaced yes)
-		(property "Reference" "#PWR032"
-			(at 48.26 71.12 0)
-			(hide yes)
-			(show_name no)
-			(do_not_autoplace no)
-			(effects
-				(font
-					(size 1.27 1.27)
-				)
-			)
-		)
-		(property "Value" "GND"
-			(at 46.99 71.12 0)
-			(show_name no)
-			(do_not_autoplace no)
-			(effects
-				(font
-					(size 1.27 1.27)
-				)
-			)
-		)
-		(property "Footprint" ""
-			(at 41.91 71.12 0)
-			(hide yes)
-			(show_name no)
-			(do_not_autoplace no)
-			(effects
-				(font
-					(size 1.27 1.27)
-				)
-			)
-		)
-		(property "Datasheet" ""
-			(at 41.91 71.12 0)
-			(hide yes)
-			(show_name no)
-			(do_not_autoplace no)
-			(effects
-				(font
-					(size 1.27 1.27)
-				)
-			)
-		)
-		(property "Description" "Power symbol creates a global label with name \"GND\" , ground"
-			(at 41.91 71.12 0)
-			(hide yes)
-			(show_name no)
-			(do_not_autoplace no)
-			(effects
-				(font
-					(size 1.27 1.27)
-				)
-			)
-		)
-		(pin "1"
-		)
-		(instances
-			(project "enclosure_pcb"
-				(path "/4a16a4d9-4fe7-4c30-8337-203b926a87e2/701ea811-00f8-4bd6-9c82-57fae78c7ace"
-					(reference "#PWR032")
-					(unit 1)
-				)
