File: pcb/_restore_backup_2026-08-16T11-09-26-026/enclosure_pcb.kicad_pcb (KiCad board)
At the start: 2 copper layers, 100 x 80 mm, 102 parts, among them J3 USB_C_Receptacle_USB2.0_14P, J4 Conn_01x03_Pin, J5 Conn_01x03_Pin, J7 Conn_01x04_Pin, J8 Conn_ARM_JTAG_SWD_10, Q1 S8050, Q2 2SC3357-T1-A, Q3 MMBT918, SW1 SW_Push_WE, SW2 SW_Lever_RSPRO_5MS1, SW3 SW_Push_WE, SW4 SW_Push_WE, U1 STM32F446RETx, U2 LD1117S33TR_SOT223, U3 LD1117S50TR_SOT223, U4 USBLC6-4SC6, U6 LM358_C5252902, Y1 Crystal_GND3, Y2 Crystal_4-pin

Commit message: feat: pcb review
Parts:
- added J6: Conn_02x12_Odd_Even, Connector_Samtec_HLE_THT:Samtec_HLE-112-02-xx-DV-TE_2x12_P2.54mm_Horizontal, F.Cu at (105.0, 90.2)
- moved J4 2.61 mm to (108.5, 101.5)
Routing:
- net +E5V: track 28.4 -> 128.9 mm
- net +U5V: track 58.2 -> 98.3 mm
- net /SCH_MCU/PUSH_BTN: track 43.7 -> 11.7 mm, vias 2 -> 0
- net +3V3: track 219.8 -> 204.4 mm, vias 0 -> 1
- net /SCH_MCU/PWM: track 28.5 -> 25.8 mm
- net /SCH_FS1000/DATA IN: track 76.7 -> 75.8 mm
- net +5V: track 181.5 -> 182.4 mm
- net /SCH_FS1000/DATA OUT: track 56.7 -> 55.9 mm
- net GND: vias 164 -> 110
